Commit message: Update collision properties for robotic arm

File: my_robot_description/urdf/arm.xacro (robot description, xacro)
@@ -20,5 +20,5 @@
                 <box size="${base_length} ${base_width} ${base_height}" />
             </geometry>
-            <origin xyz="0 0 0" rpy="0 0 0" />
+            <origin xyz="0 0 ${base_height / 2.0}" rpy="0 0 0" />
         </collision>
         <xacro:box_inertia m="0.5" x="${base_length}" y="${base_width}" z="${base_height}"
@@ -51,10 +51,5 @@
         <origin xyz="0 0 ${base_height / 2.0}" rpy="0 0 0" />
         <axis xyz="0 1 0" />
-        <limit
-            lower="0"
-            upper="${pi/2.0}"
-            effort="100"
-            velocity="100"
-        />
+        <limit lower="0" upper="${pi/2.0}" effort="100" velocity="100" />
         <dynamics friction="0.3" damping="0.3" />
     </joint>
@@ -64,10 +59,5 @@
         <origin xyz="0 0 ${arm_length}" rpy="0 0 0" />
         <axis xyz="0 1 0" />
-        <limit
-            lower="0"
-            upper="${pi/2.0}"
-            effort="100"
-            velocity="100"
-        />
+        <limit lower="0" upper="${pi/2.0}" effort="100" velocity="100" />
         <dynamics friction="0.3" damping="0.3" />
     </joint>

Commit message: Added comment for friction properties

File: my_robot_description/urdf/arm.xacro (robot description, xacro)
@@ -52,5 +52,5 @@
         <axis xyz="0 1 0" />
         <limit lower="0" upper="${pi/2.0}" effort="100" velocity="100" />
-        <dynamics friction="0.3" damping="0.3" />
+        <dynamics friction="0.3" damping="0.3" /> <!-- We add these friction elements to avoid the robotic arm to fall directly due to an umbalance in Gazebo -->
     </joint>
     <joint name="forearm_hand_joint" type="revolute">
