Commit message: Add Final Project Development

File: my_robot_description/urdf/mobile_base.xacro (robot description, xacro)
@@ -81,3 +81,8 @@
         <origin xyz="${base_length / 3.0} 0 ${-wheel_radius / 2.0}" rpy="0 0 0" />
     </joint>
+    <joint name="base_arm_base_link" type="fixed">
+        <parent link="base_link" />
+        <child link="arm_base_link" />
+        <origin xyz="0 0 ${base_height}" rpy="0 0 0" />
+    </joint>
 </robot>

File: my_robot_description/urdf/mobile_base_gazebo.xacro (robot description, xacro)
@@ -23,7 +23,25 @@
             filename="gz-sim-joint-state-publisher-system"
             name="gz::sim::systems::JointStatePublisher">
+            <joint_name>base_left_wheel_joint</joint_name>
+            <joint_name>base_right_wheel_joint</joint_name>
+            <joint_name>arm_base_forearm_joint</joint_name>
+            <joint_name>forearm_hand_joint</joint_name>
         </plugin>
-        <joint_name>base_left_wheel_joint</joint_name>
-        <joint_name>base_right_wheel_joint</joint_name>
+    </gazebo>
+    <gazebo>
+        <plugin
+            filename="gz-sim-joint-position-controller-system"
+            name="gz::sim::systems::JointPositionController">
+            <joint_name>arm_base_forearm_joint</joint_name>
+            <p_gain>5.0</p_gain>
+        </plugin>
+    </gazebo>
+    <gazebo>
+        <plugin
+            filename="gz-sim-joint-position-controller-system"
+            name="gz::sim::systems::JointPositionController">
+            <joint_name>forearm_hand_joint</joint_name>
+            <p_gain>3.0</p_gain>
+        </plugin>
     </gazebo>
 </robot>

File: my_robot_description/urdf/my_robot.urdf.xacro (robot description, xacro)
@@ -2,4 +2,5 @@
 <robot name="my_robot" xmlns:xacro="http://www.ros.org/wiki/xacro"> <!-- Aqui ponemos el nombre del robot, cómo lo queramos llamar -->
     <xacro:include filename="common_properties.xacro" />
+    <xacro:include filename="arm.xacro" />
     <xacro:include filename="mobile_base.xacro" />
     <xacro:include filename="mobile_base_gazebo.xacro" />

File: robot_arm_description/urdf/common_properties.xacro (robot description, xacro)
@@ -1,13 +1,4 @@
 <?xml version="1.0"?>
 <robot xmlns:xacro="http://www.ros.org/wiki/xacro">
-    <material name="blue">
-        <color rgba="0 0 0.5 1" />
-    </material>
-    <material name="grey">
-        <color rgba="0.5 0.5 0.5 1" />
-    </material>
-    <material name="red">
-        <color rgba="0.8 0 0 1" />
-    </material>
     <material name="yellow">
         <color rgba="1 1 0 1" />
@@ -34,11 +25,3 @@
         </inertial>
     </xacro:macro>
-    <xacro:macro name="sphere_inertia" params="m r"> <!--The inertia formula of a solid sphere is used in this case, instead of a hollow sphere-->
-        <inertial>
-            <mass value="${m}" />
-            <inertia ixx="${(2*m/5) * (r*r)}" ixy="0" ixz="0"
-                     iyy="${(2*m/5) * (r*r)}" iyz="0"
-                     izz="${(2*m/5) * (r*r)}" />
-        </inertial>
-    </xacro:macro>
 </robot>

Commit message: Adding modification from URDF file

File: my_robot_description/urdf/mobile_base.xacro (robot description, xacro)
@@ -84,5 +84,5 @@
         <parent link="base_link" />
         <child link="arm_base_link" />
-        <origin xyz="0 0 ${base_height}" rpy="0 0 0" />
+        <origin xyz="${base_length / 4.0} 0 ${base_height}" rpy="0 0 0" />
     </joint>
 </robot>
